File: pcb/Project-H10.sch (EAGLE design)
At the start: 0 parts

Commit message: Add component libs
Parts:
- added J1: 03JQ-STCONN_03JQ-ST_JST, Project-H10:03JQ-STCONN_03JQ-ST_JST
- added J2: PJ-609BA, Project-H10:PJ-609BA
- added U1: STM32U575VIT6LQFP-100_STM, Project-H10:STM32U575VIT6LQFP-100_STM
Connections:
- new net N$1: J1.1, J2.1
- new net N$2: J1.2, J2.3
- new net N$3: J1.3, J2.2
Other:
- note added: "Phone Jack Riser"
Changed lines of the file:
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@@
 <grid distance="0.1" unitdist="inch" unit="inch" style="lines" multiple="1" display="yes" altdistance="0.01" altunitdist="inch" altunit="inch"/>
 <layers>
+<layer number="1" name="Top" color="4" fill="1" visible="no" active="no"/>
+<layer number="2" name="Route2" color="16" fill="1" visible="no" active="no"/>
+<layer number="3" name="Route3" color="17" fill="1" visible="no" active="no"/>
+<layer number="4" name="Route4" color="18" fill="1" visible="no" active="no"/>
+<layer number="5" name="Route5" color="19" fill="1" visible="no" active="no"/>
+<layer number="6" name="Route6" color="25" fill="1" visible="no" active="no"/>
+<layer number="7" name="Route7" color="26" fill="1" visible="no" active="no"/>
+<layer number="8" name="Route8" color="27" fill="1" visible="no" active="no"/>
+<layer number="9" name="Route9" color="28" fill="1" visible="no" active="no"/>
+<layer number="10" name="Route10" color="29" fill="1" visible="no" active="no"/>
+<layer number="11" name="Route11" color="30" fill="1" visible="no" active="no"/>
+<layer number="12" name="Route12" color="20" fill="1" visible="no" active="no"/>
+<layer number="13" name="Route13" color="21" fill="1" visible="no" active="no"/>
+<layer number="14" name="Route14" color="22" fill="1" visible="no" active="no"/>
+<layer number="15" name="Route15" color="23" fill="1" visible="no" active="no"/>
+<layer number="16" name="Bottom" color="1" fill="1" visible="no" active="no"/>
+<layer number="17" name="Pads" color="2" fill="1" visible="no" active="no"/>
+<layer number="18" name="Vias" color="2" fill="1" visible="no" active="no"/>
+<layer number="19" name="Unrouted" color="6" fill="1" visible="no" active="no"/>
+<layer number="20" name="Dimension" color="24" fill="1" visible="no" active="no"/>
+<layer number="21" name="tPlace" color="7" fill="1" visible="no" active="no"/>
+<layer number="22" name="bPlace" color="7" fill="1" visible="no" active="no"/>
+<layer number="23" name="tOrigins" color="15" fill="1" visible="no" active="no"/>
+<layer number="24" name="bOrigins" color="15" fill="1" visible="no" active="no"/>
+<layer number="25" name="tNames" color="7" fill="1" visible="no" active="no"/>
+<layer number="26" name="bNames" color="7" fill="1" visible="no" active="no"/>
+<layer number="27" name="tValues" color="7" fill="1" visible="no" active="no"/>
+<layer number="28" name="bValues" color="7" fill="1" visible="no" active="no"/>
+<layer number="29" name="tStop" color="7" fill="3" visible="no" active="no"/>
+<layer number="30" name="bStop" color="7" fill="6" visible="no" active="no"/>
+<layer number="31" name="tCream" color="7" fill="4" visible="no" active="no"/>
+<layer number="32" name="bCream" color="7" fill="5" visible="no" active="no"/>
+<layer number="33" name="tFinish" color="6" fill="3" visible="no" active="no"/>
+<layer number="34" name="bFinish" color="6" fill="6" visible="no" active="no"/>
+<layer number="35" name="tGlue" color="7" fill="4" visible="no" active="no"/>
+<layer number="36" name="bGlue" color="7" fill="5" visible="no" active="no"/>
+<layer number="37" name="tTest" color="7" fill="1" visible="no" active="no"/>
+<layer number="38" name="bTest" color="7" fill="1" visible="no" active="no"/>
+<layer number="39" name="tKeepout" color="4" fill="11" visible="no" active="no"/>
+<layer number="40" name="bKeepout" color="1" fill="11" visible="no" active="no"/>
+<layer number="41" name="tRestrict" color="4" fill="10" visible="no" active="no"/>
+<layer number="42" name="bRestrict" color="1" fill="10" visible="no" active="no"/>
+<layer number="43" name="vRestrict" color="2" fill="10" visible="no" active="no"/>
+<layer number="44" name="Drills" color="7" fill="1" visible="no" active="no"/>
+<layer number="45" name="Holes" color="7" fill="1" visible="no" active="no"/>
+<layer number="46" name="Milling" color="3" fill="1" visible="no" active="no"/>
+<layer number="47" name="Measures" color="7" fill="1" visible="no" active="no"/>
+<layer number="48" name="Document" color="7" fill="1" visible="no" active="no"/>
+<layer number="49" name="Reference" color="7" fill="1" visible="no" active="no"/>
+<layer number="51" name="tDocu" color="7" fill="1" visible="no" active="no"/>
+<layer number="52" name="bDocu" color="7" fill="1" visible="no" active="no"/>
 <layer number="88" name="SimResults" color="9" fill="1" visible="yes" active="yes"/>
 <layer number="89" name="SimProbes" color="9" fill="1" visible="yes" active="yes"/>
@@
 </classes>
 <parts>
+<part name="U1" library="Project-H10" deviceset="STM32U575VIT6" device="LQFP-100_STM"/>
+<part name="J1" library="Project-H10" deviceset="03JQ-ST" device="CONN_03JQ-ST_JST"/>
+<part name="J2" library="Project-H10" deviceset="PJ-609BA" device=""/>
 </parts>
 <sheets>
 <sheet>
 <plain>
+<text x="-58.42" y="-30.48" size="2.54" layer="97">Phone Jack Riser</text>
 </plain>
 <instances>
+<instance part="U1" gate="A" x="10.16" y="81.28" smashed="yes">
+<attribute name="NAME" x="18.1346" y="90.3986" size="2.083" layer="95" ratio="6"/>
+<attribute name="VALUE" x="17.4952" y="87.8586" size="2.083" layer="96" ratio="6"/>
+</instance>
+<instance part="U1" gate="B" x="86.36" y="76.2" smashed="yes">
+<attribute name="NAME" x="94.3346" y="85.3186" size="2.083" layer="95" ratio="6"/>
+<attribute name="VALUE" x="93.6952" y="82.7786" size="2.083" layer="96" ratio="6"/>
+</instance>
+<instance part="U1" gate="C" x="88.9" y="15.24" smashed="yes">
+<attribute name="NAME" x="96.8746" y="24.3586" size="2.083" layer="95" ratio="6"/>
+<attribute name="VALUE" x="96.2352" y="21.8186" size="2.083" layer="96" ratio="6"/>
+</instance>
+<instance part="J1" gate="A" x="-45.72" y="-45.72" smashed="yes" rot="R180">
+<attribute name="NAME" x="-55.4726" y="-35.2806" size="2.083" layer="95" ratio="6" rot="R180"/>
+</instance>
+<instance part="J2" gate="G$1" x="-30.48" y="-40.64" smashed="yes">
+<attribute name="NAME" x="-33.02" y="-36.576" size="1.778" layer="95"/>
+<attribute name="VALUE" x="-33.02" y="-49.53" size="1.778" layer="96"/>
+</instance>
 </instances>
 <busses>
 </busses>
 <nets>
+<net name="N$1" class="0">
+<segment>
+<pinref part="J2" gate="G$1" pin="1"/>
+<pinref part="J1" gate="A" pin="1"/>
+<wire x1="-35.56" y1="-45.72" x2="-45.72" y2="-45.72" width="0.1524" layer="91"/>
+</segment>
+</net>
+<net name="N$2" class="0">
+<segment>
+<pinref part="J2" gate="G$1" pin="3"/>
+<pinref part="J1" gate="A" pin="2"/>
+<wire x1="-35.56" y1="-43.18" x2="-45.72" y2="-43.18" width="0.1524" layer="91"/>
+</segment>
+</net>
+<net name="N$3" class="0">
+<segment>
+<pinref part="J1" gate="A" pin="3"/>
+<wire x1="-45.72" y1="-40.64" x2="-38.1" y2="-40.64" width="0.1524" layer="91"/>
+<wire x1="-38.1" y1="-40.64" x2="-38.1" y2="-38.1" width="0.1524" layer="91"/>
+<pinref part="J2" gate="G$1" pin="2"/>
+<wire x1="-38.1" y1="-38.1" x2="-35.56" y2="-38.1" width="0.1524" layer="91"/>
+</segment>
+</net>
 </nets>
 </sheet>
