File: pcb/Project-H10.sch (EAGLE design)
At the start: 3 parts, among them J1 03JQ-STCONN_03JQ-ST_JST, J2 PJ-609BA, U1 STM32U575VIT6LQFP-100_STM

Commit message: replace buf output stage
Parts:
- added J3, J4: 08JQ-BT, Project-H10:08JQ-BT
- added J5: B3B-XH-A(LF)(SN)CONN_B3B-XH-A_JST, Project-H10:B3B-XH-A(LF)(SN)CONN_B3B-XH-A_JST
- added J6, J7: B8B-XH-A, Project-H10:B8B-XH-A_(LF)(SN)CONN_B8B-XH-A_JST
- added U10, U9: LM1972MX/NOPBM20B_TEX, Project-H10:LM1972MX/NOPBM20B_TEX
- added U2: CS4398-CZZCIR-TSSOP-28, Project-H10:CS4398-CZZCIR-TSSOP-28
- added U3: CS8416-CZZCIR-TSSOP-28, Project-H10:CS8416-CZZCIR-TSSOP-28
- added U4: OPA2228P, Project-H10:OPAMP2
- added U5, U6, U7, U8: NJM4556AD, Project-H10:OPAMP2
- J1: value 03JQ-STCONN_03JQ-ST_JST -> 03JQ-ST
Connections:
- net N$1 renamed PH_COM
- net N$2 renamed PH_R
- net N$3 renamed PH_L
Other:
- note added: "DAC Module"
- note added: "HP Amplifier"
- note added: "SPDIF Decoder"
- moved on the sheet: J1, J2, U1A, U1B, U1C
